File: PCB_Gafas/PCB_Glasses/PCB_Glasses.kicad_sch (KiCad schematic)
At the start: 11 parts, among them J1 Conn_01x02_Socket, J2 Conn_01x04_Socket, J3 Conn_01x04_Socket, J4 Conn_01x02_Socket, SW1 SW_Push, U1 XIAO ESP32C3, U2 module_mpu6050

Commit message: Cosa
Parts:
- removed J3: Conn_01x04_Socket, Connector_JST:JST_EH_B4B-EH-A_1x04_P2.50mm_Vertical, symbol Connector:Conn_01x04_Socket
- SW1: footprint Button_Switch_SMD:SW_SPST_PTS645 -> Button_Switch_SMD:SW_SPST_CK_RS282G05A3
