File: PCB_Gafas/PCB_Glasses/PCB_Glasses.kicad_pcb (KiCad board)
At the start: 2 copper layers, 10 parts, among them J1 Conn_01x02_Socket, J2 Conn_01x04_Socket, J3 Conn_01x04_Socket, J4 Conn_01x02_Socket, U1 XIAO ESP32C3, U2 module_mpu6050

Commit message: Started Gafas Routing
Parts:
- removed J3: Conn_01x04_Socket, Connector_JST:JST_EH_B4B-EH-A_1x04_P2.50mm_Vertical
- added SW1: SW_Push, Button_Switch_SMD:SW_SPST_CK_RS282G05A3, F.Cu at (54.8, 29.5)
- R1, R2: value 220k -> 22k
- moved R1 47.2 mm to (23.6, 44.0)
- moved R2 47.0 mm to (23.3, 49.2)
- moved R3 44.5 mm to (39.5, 29.2), turned to 180 degrees
- moved D1 42.6 mm to (46.2, 29.2), turned to 180 degrees
- moved J1 41.6 mm to (23.2, 37.8), turned to 90 degrees
- moved J2 36.4 mm to (64.2, 29.2)
- moved U1 32.3 mm to (37.7, 39.3), turned to 180 degrees
- moved J4 26.7 mm to (77.0, 41.8), turned to -90 degrees
- moved U2 23.9 mm to (54.5, 34.5), turned to -90 degrees
Connections:
- U1 pad 7: unconnected-(U1-D6-Pad7) -> Net-(U1-D6)
- U2 pad 7: unconnected-(U2-ADD-Pad7) -> GND
Routing:
- net /SDA: track 0.00 -> 27.3 mm
- net /SCL: track 0.00 -> 21.3 mm
- added copper zone on B.Cu, net GND
Other:
- board outline added: 60 x 25 mm

Commit message: PCB Glasses Done
Parts:
- moved SW1 0.32 mm to (54.6, 29.2)
- moved R1 0.19 mm to (23.6, 43.8)
Routing:
- net +3V8: track 0.00 -> 54.8 mm
- net +3.3V: track 0.00 -> 45.2 mm, vias 0 -> 1
- net /D1: track 0.00 -> 31.5 mm
- net /D2: track 0.00 -> 31.5 mm
- net Net-(U1-D3): track 0.00 -> 15.7 mm
- net Net-(U1-D6): track 0.00 -> 8.12 mm
- net /SCL: track 21.3 -> 29.4 mm, vias 0 -> 1
- net Net-(U1-D0): track 0.00 -> 5.54 mm
- net Net-(D1-A): track 0.00 -> 4.26 mm
Other:
- outline, holes or cut-outs redrawn

Commit message: Finales
Parts:
- moved R2 1.62 mm to (23.3, 47.6)
Routing:
- net Net-(U1-D0): track 5.54 -> 31.3 mm
- added copper zone on F.Cu, net GND
Other:
- board text added: "FGA| 2025"
Changed lines of the file:
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@@
 		)
 		(property "Footprint" "XIAO_ESP32C3-main:xiao_esp32c3"
-			(at 0 0 360)
+			(at 0 0 0)
 			(layer "F.Fab")
 			(hide yes)
@@
 		)
 		(property "Datasheet" "https://files.seeedstudio.com/wiki/Seeed-Studio-XIAO-ESP32/esp32-c3_datasheet.pdf"
-			(at 0 0 360)
+			(at 0 0 0)
 			(layer "F.Fab")
 			(hide yes)
@@
 		)
 		(property "Description" "ESP32C3 Transceiver Evaluation Board"
-			(at 0 0 360)
+			(at 0 0 0)
 			(layer "F.Fab")
 			(hide yes)
@@
 		(tags "LED")
 		(property "Reference" "D1"
-			(at 0 -1.65 360)
+			(at 0 -1.65 0)
 			(layer "F.SilkS")
 			(effects
@@
 		)
 		(property "Value" "LED"
-			(at 0 1.65 360)
+			(at 0 1.65 0)
 			(layer "F.Fab")
 			(effects
@@
 		)
 		(fp_text user "${REFERENCE}"
-			(at 0 0 360)
+			(at 0 0 0)
 			(layer "F.Fab")
 			(effects
@@
 	(footprint "Resistor_SMD:R_1206_3216Metric_Pad1.30x1.75mm_HandSolder"
 		(layer "F.Cu")
-		(at 23.3 49.25)
+		(at 23.3 47.625)
 		(descr "Resistor SMD 1206 (3216 Metric), square (rectangular) end terminal, IPC_7351 nominal with elongated pad for handsoldering. (Body size source: IPC-SM-782 page 72, https://www.pcb-3d.com/wordpress/wp-content/uploads/ipc-sm-782a_amendment_1_and_2.pdf), generated with kicad-footprint-generator")
 		(tags "resistor handsolder")
@@
 		(tags "connector JST EH vertical")
 		(property "Reference" "J2"
-			(at 3.75 -2.8 360)
+			(at 3.75 -2.8 0)
 			(layer "F.SilkS")
 			(effects
@@
 		)
 		(property "Value" "Conn_01x04_Socket"
-			(at 3.75 3.4 360)
+			(at 3.75 3.4 0)
 			(layer "F.Fab")
 			(effects
@@
 		)
 		(fp_text user "${REFERENCE}"
-			(at 3.75 1.5 360)
+			(at 3.75 1.5 0)
 			(layer "F.Fab")
 			(effects
@@
 		(tags "resistor handsolder")
 		(property "Reference" "R3"
-			(at 0 -1.82 360)
+			(at 0 -1.82 0)
 			(layer "F.SilkS")
 			(effects
@@
 		)
 		(property "Value" "130"
-			(at 0 1.82 360)
+			(at 0 1.82 0)
 			(layer "F.Fab")
 			(effects
@@
 		)
 		(fp_text user "${REFERENCE}"
-			(at 0 0 360)
+			(at 0 0 0)
 			(layer "F.Fab")
 			(effects
@@
 		(layer "Edge.Cuts")
 	)
+	(gr_text "FGA|\n2025"
+		(at 26.67 31.115 0)
+		(layer "F.SilkS")
+		(effects
+			(font
+				(size 1.5 1.5)
+				(thickness 0.15)
+			)
+			(justify left bottom)
+		)
+	)
 	(segment
 		(start 41.05 29.25)
@@
 	(via
 		(at 60.96 36.83)
-		(size 0.6)
-		(drill 0.3)
+		(size 1.27)
+		(drill 0.6)
 		(layers "F.Cu" "B.Cu")
 		(net 5)
@@
 	(via
 		(at 36.195 41.91)
-		(size 0.6)
-		(drill 0.3)
+		(size 1.27)
+		(drill 0.6)
 		(layers "F.Cu" "B.Cu")
 		(net 6)
@@
 	)
 	(segment
-		(start 21.75 49.25)
-		(end 21.75 44.065)
+		(start 41.43 48.74)
+		(end 46.275 48.74)
+		(width 0.5)
+		(layer "F.Cu")
+		(net 9)
+	)
+	(segment
+		(start 22 47.375)
+		(end 21.75 47.625)
+		(width 0.5)
+		(layer "F.Cu")
+		(net 9)
+	)
+	(segment
+		(start 21.75 49.055)
+		(end 22.86 50.165)
 		(width 0.5)
 		(layer "F.Cu")
@@
 	)
 	(segment
+		(start 22.86 50.165)
+		(end 40.005 50.165)
+		(width 0.5)
+		(layer "F.Cu")
+		(net 9)
+	)
+	(segment
+		(start 40.005 50.165)
+		(end 41.43 48.74)
+		(width 0.5)
+		(layer "F.Cu")
+		(net 9)
+	)
+	(segment
+		(start 21.75 47.625)
+		(end 21.75 49.055)
+		(width 0.5)
+		(layer "F.Cu")
+		(net 9)
+	)
+	(segment
+		(start 22 43.815)
+		(end 22 47.375)
+		(width 0.5)
+		(layer "F.Cu")
+		(net 9)
+	)
+	(segment
 		(start 46.275 41.12)
 		(end 45.565 41.12)
@@
 	)
 	(zone
+		(net 1)
+		(net_name "GND")
+		(layer "F.Cu")
+		(hatch edge 0.5)
+		(priority 1)
+		(connect_pads
+			(clearance 0.5)
+		)
+		(min_thickness 0.25)
+		(filled_areas_thickness no)
+		(fill yes
+			(thermal_gap 0.5)
+			(thermal_bridge_width 0.5)
+		)
+		(polygon
+			(pts
+				(xy 20.32 26.67) (xy 20.32 50.8) (xy 79.375 50.8) (xy 79.375 26.67)
+			)
+		)
+	)
+	(zone
