File: PCB_Fuente/Fuente_Final/Fuente_Final.kicad_pcb (KiCad board)
At the start: 2 copper layers, 58.8 x 32.5 mm, 14 parts, among them J1 Conn_01x02_Socket, J2 USB_A, J3 Conn_01x02_Socket, J4 USB_A, T1 Transformer_1P_1S, U1 L7805

Commit message: Finales
Parts:
- moved J3 3.19 mm to (20.3, 38.7)
Routing:
- net Net-(J3-Pin_2): track 7.55 -> 10.8 mm
- net Net-(J3-Pin_1): track 8.00 -> 11.1 mm
Other:
- board size 58.8 x 32.5 mm -> 62.4 x 32.5 mm
- board text added: "Do Not Feed the Capacitors"
- board text added: "FGA | 2025"
Changed lines of the file:
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@@
 			(outputformat 1)
 			(mirror no)
-			(drillshape 1)
+			(drillshape 0)
 			(scaleselection 1)
-			(outputdirectory "")
+			(outputdirectory "Fabrication/")
 		)
 	)
@@
 		(tags "Diode DO-15 series Axial Vertical pin pitch 5.08mm  length 7.6mm diameter 3.6mm")
 		(property "Reference" "D3"
-			(at 2.54 -2.92 360)
+			(at 2.54 -2.92 0)
 			(layer "F.SilkS")
 			(effects
@@
 		)
 		(property "Value" "D_45deg"
-			(at 2.54 2.92 360)
+			(at 2.54 2.92 0)
 			(layer "F.Fab")
 			(effects
@@
 		)
 		(fp_text user "A"
-			(at 3.18 1.2 360)
+			(at 3.18 1.2 0)
 			(layer "F.SilkS")
 			(effects
@@
 		)
 		(fp_text user "A"
-			(at 3.18 1.2 360)
+			(at 3.18 1.2 0)
 			(layer "F.Fab")
 			(effects
@@
 		)
 		(fp_text user "${REFERENCE}"
-			(at 2.54 -2.92 360)
+			(at 2.54 -2.92 0)
 			(layer "F.Fab")
 			(effects
@@
 		(tags "LED handsolder")
 		(property "Reference" "D5"
-			(at 0 -1.65 360)
+			(at 0 -1.65 0)
 			(layer "F.SilkS")
 			(effects
@@
 		)
 		(property "Value" "LED"
-			(at 0 1.65 360)
+			(at 0 1.65 0)
 			(layer "F.Fab")
 			(effects
@@
 		)
 		(fp_text user "${REFERENCE}"
-			(at 0 0 360)
+			(at 0 0 0)
 			(layer "F.Fab")
 			(effects
@@
 		(tags "Diode DO-15 series Axial Vertical pin pitch 5.08mm  length 7.6mm diameter 3.6mm")
 		(property "Reference" "D2"
-			(at 2.54 -2.92 360)
+			(at 2.54 -2.92 0)
 			(layer "F.SilkS")
 			(effects
@@
 		)
 		(property "Value" "D_45deg"
-			(at 2.54 2.92 360)
+			(at 2.54 2.92 0)
 			(layer "F.Fab")
 			(effects
@@
 		)
 		(fp_text user "K"
-			(at 1.9 1.2 360)
+			(at 1.9 1.2 0)
 			(layer "F.SilkS")
 			(effects
@@
 		)
 		(fp_text user "K"
-			(at 1.9 1.2 360)
+			(at 1.9 1.2 0)
 			(layer "F.Fab")
 			(effects
@@
 		)
 		(fp_text user "${REFERENCE}"
-			(at 2.54 -2.92 360)
+			(at 2.54 -2.92 0)
 			(layer "F.Fab")
 			(effects
@@
 		(tags "Diode DO-15 series Axial Vertical pin pitch 5.08mm  length 7.6mm diameter 3.6mm")
 		(property "Reference" "D1"
-			(at 2.54 -2.92 360)
+			(at 2.54 -2.92 0)
 			(layer "F.SilkS")
 			(effects
@@
 		)
 		(property "Value" "D_45deg"
-			(at 2.54 2.92 360)
+			(at 2.54 2.92 0)
 			(layer "F.Fab")
 			(effects
@@
 		)
 		(fp_text user "A"
-			(at 3.18 1.2 360)
+			(at 3.18 1.2 0)
 			(layer "F.SilkS")
 			(effects
@@
 		)
 		(fp_text user "${REFERENCE}"
-			(at 2.54 -2.92 360)
+			(at 2.54 -2.92 0)
 			(layer "F.Fab")
 			(effects
@@
 		)
 		(fp_text user "A"
-			(at 3.18 1.2 360)
+			(at 3.18 1.2 0)
 			(layer "F.Fab")
 			(effects
@@
 	(footprint "TerminalBlock:TerminalBlock_bornier-2_P5.08mm"
 		(layer "F.Cu")
-		(at 23.5 38.5 90)
+		(at 20.32 38.735 90)
 		(descr "simple 2-pin terminal block, pitch 5.08mm, revamped version of bornier2")
 		(tags "terminal block bornier2")
@@
 		(tags "resistor handsolder")
 		(property "Reference" "R1"
-			(at 0 -1.65 360)
+			(at 0 -1.65 0)
 			(layer "F.SilkS")
 			(effects
@@
 		)
 		(property "Value" "R"
-			(at 0 1.65 360)
+			(at 0 1.65 0)
 			(layer "F.Fab")
 			(effects
@@
 		)
 		(fp_text user "${REFERENCE}"
-			(at 0 0 360)
+			(at 0 0 0)
 			(layer "F.Fab")
 			(effects
@@
 		(tags "connector JST EH vertical")
 		(property "Reference" "J1"
-			(at 1.25 -2.8 360)
+			(at 1.25 -2.8 0)
 			(layer "F.SilkS")
 			(effects
@@
 		)
 		(property "Value" "Conn_01x02_Socket"
-			(at -0.05 13.8 360)
+			(at -0.05 13.8 0)
 			(layer "F.Fab")
 			(effects
@@
 		)
 		(fp_text user "${REFERENCE}"
-			(at 1.25 1.5 360)
+			(at 1.25 1.5 0)
 			(layer "F.Fab")
 			(effects
@@
 		(tags "Diode DO-15 series Axial Vertical pin pitch 5.08mm  length 7.6mm diameter 3.6mm")
 		(property "Reference" "D4"
-			(at 2.54 -2.92 360)
+			(at 2.54 -2.92 0)
 			(layer "F.SilkS")
 			(effects
@@
 		)
 		(property "Value" "D_45deg"
-			(at 2.54 2.92 360)
+			(at 2.54 2.92 0)
 			(layer "F.Fab")
 			(effects
@@
 		)
 		(fp_text user "K"
-			(at 1.9 1.2 360)
+			(at 1.9 1.2 0)
 			(layer "F.SilkS")
 			(effects
@@
 		)
 		(fp_text user "K"
-			(at 1.9 1.2 360)
+			(at 1.9 1.2 0)
 			(layer "F.Fab")
 			(effects
@@
 		)
 		(fp_text user "${REFERENCE}"
-			(at 2.54 -2.92 360)
+			(at 2.54 -2.92 0)
 			(layer "F.Fab")
 			(effects
@@
 	)
 	(gr_line
-		(start 19.25 20.5)
-		(end 19.5 53)
+		(start 15.625 20.5)
+		(end 15.875 53)
 		(stroke
 			(width 0.05)
@@
 	)
 	(gr_line
-		(start 19.5 53)
+		(start 15.875 53)
 		(end 74.5 53)
 		(stroke
@@
 	(gr_line
 		(start 74.25 20.5)
-		(end 19.25 20.5)
+		(end 15.625 20.5)
 		(stroke
 			(width 0.05)
@@
 		(layer "Edge.Cuts")
 	)
+	(gr_text "Do Not Feed \nthe Capacitors"
+		(at 41.91 29.845 0)
+		(layer "F.SilkS")
+		(effects
+			(font
+				(size 1 1)
+				(thickness 0.25)
+				(bold yes)
+			)
+			(justify left bottom)
+		)
+	)
+	(gr_text "FGA | 2025"
+		(at 49.53 51.435 0)
+		(layer "F.SilkS")
+		(effects
+			(font
+				(size 1.5 1.5)
+				(thickness 0.2)
+			)
+			(justify left bottom)
+		)
+	)
 	(segment
 		(start 32.16 31.5)
@@
 	)
 	(segment
+		(start 20.555 33.42)
+		(end 29.04 33.42)
+		(width 0.5)
+		(layer "F.Cu")
+		(net 8)
+	)
+	(segment
 		(start 29.04 33.42)
 		(end 30.46 32)
@@
 	)
 	(segment
-		(start 23.5 33.42)
-		(end 29.04 33.42)
+		(start 20.32 33.655)
+		(end 20.555 33.42)
 		(width 0.5)
 		(layer "F.Cu")
@@
 	)
 	(segment
-		(start 27.96 38.5)
+		(start 20.32 38.735)
+		(end 24.765 38.735)
+		(width 0.5)
+		(layer "F.Cu")
+		(net 9)
+	)
+	(segment
+		(start 27.03 41)
 		(end 30.46 41)
 		(width 0.5)
@@
 	)
 	(segment
-		(start 23.5 38.5)
-		(end 27.96 38.5)
+		(start 24.765 38.735)
+		(end 27.03 41)
 		(width 0.5)
 		(layer "F.Cu")
@@
 		(polygon
 			(pts
-				(xy 19.5 20.5) (xy 19.5 53) (xy 74 53) (xy 74.25 20.5)
+				(xy 15.875 20.5) (xy 15.875 53) (xy 74 53) (xy 74.25 20.5)
 			)
 		)
