File: PCB_Pecho/PCB_pecho/PCB_pecho.kicad_sch (KiCad schematic)
At the start: 2 parts, among them U1 ESP32-S3-DEVKITC-1-N8R2, U2 module_mpu6050

Commit message: Finales
Parts:
- added J1, J7: Conn_01x04_Pin, Connector_JST:JST_EH_B4B-EH-A_1x04_P2.50mm_Vertical, symbol Connector:Conn_01x04_Pin
- added J2: Conn_01x02_Socket, Connector_JST:JST_EH_B2B-EH-A_1x02_P2.50mm_Vertical, symbol Connector:Conn_01x02_Socket
- added J3, J4, J5, J6: Conn_01x04_Socket, Connector_JST:JST_EH_B4B-EH-A_1x04_P2.50mm_Vertical, symbol Connector:Conn_01x04_Socket
- added R1: 10k, Resistor_SMD:R_1206_3216Metric_Pad1.30x1.75mm_HandSolder, symbol Device:R
- added U3: module_bme280, usini_sensors:module_bme280, symbol usini_sensors:module_bme280
- added U4: ~, symbol XL6009_Boost_Module:BoostConvXL6009_Boost_Module
Connections:
- net GND: now also U2.2 (GND), J3.2 (Pin_2), J4.2 (Pin_2), J5.2 (Pin_2), J6.1 (Pin_1), J6.2 (Pin_2), J7.1 (Pin_1), J7.2 (Pin_2), J7.3 (Pin_3), J7.4 (Pin_4), R1.1, U3.2 (GND), U4.2 (IN-), U4.4 (OUT-)
- net +5V: now reaches U2.1 (VCC)
- net +5V: now also U1.J1_21 (5V0), J3.1 (Pin_1), J5.1 (Pin_1), U4.3 (OUT+)
- net SCL: now reaches U2.3 (SCL)
- net SCL: now also U1.J1_15 (GPIO9), J3.4 (Pin_4), J4.4 (Pin_4), J5.4 (Pin_4), U3.3 (SCL)
- net SDA: now reaches U2.4 (SDA)
- net SDA: now also U1.J1_12 (GPIO8), J3.3 (Pin_3), J4.3 (Pin_3), J5.3 (Pin_3), U3.4 (SDA)
- net +3.3V: now reaches U1.J1_1 (3V3), U1.J1_2 (3V3)
- net +3.3V: now also J2.2 (Pin_2), J4.1 (Pin_1), U3.1 (VCC)
- net D1: now reaches U1.J1_19 (GPIO13)
- net D1: now also J1.4 (Pin_4)
- net D2: now reaches U1.J1_20 (GPIO14)
- net D2: now also J1.3 (Pin_3)
- net D3: now reaches U1.J1_8 (GPIO15)
- net D3: now also J1.2 (Pin_2)
- net D4: now reaches U1.J1_9 (GPIO16)
- net D4: now also J1.1 (Pin_1)
- net at U1.J3_14 (GPIO0): now also J2.1 (Pin_1), R1.2
- new net +4V: J6.3 (Pin_3), J6.4 (Pin_4), U4.1 (IN+)
- no-connect marks 0 -> 6
Other:
- moved on the sheet: U2
